Commit message: filter velocity control

File: my_pybullet_envs/assets/cylinder_heavier.urdf (robot description, URDF)
Before this commit: robot urdf_robot, 1 links, 0 joints
Links:
- link baseLink: mass 10.0 -> 5.0

Commit message: mods and refactors, see notes

File: my_pybullet_envs/assets/cylinder_heavier.urdf (robot description, URDF)
Before this commit: robot urdf_robot, 1 links, 0 joints
Links:
- link baseLink: mass 5.0 -> 2.5
