Commit message: revert shadow hand grasping 1208

File: my_pybullet_envs/assets/box.urdf (robot description, URDF)
Before this commit: robot tabletop, 1 links, 0 joints
Links:
- link baseLink: mass 5.0 -> 2.0; geometry collision box size=0.08 0.08 0.18; visual box size=0.08 0.08 0.18

File: my_pybullet_envs/assets/cylinder_heavier.urdf (robot description, URDF)
Before this commit: robot urdf_robot, 1 links, 0 joints
Links:
- link baseLink: mass 2.5 -> 2.0

Commit message: box grasping easy seed14

File: my_pybullet_envs/assets/box.urdf (robot description, URDF)
Before this commit: robot urdf_robot, 1 links, 0 joints
Links:
- link baseLink: mass 2.0 -> 3.5

File: my_pybullet_envs/assets/cylinder.urdf (robot description, URDF)
Before this commit: robot urdf_robot, 1 links, 0 joints
Links:
- link baseLink: mass 5.0 -> 3.5
