Commit message: no cylinder state

File: my_pybullet_envs/assets/cylinder.urdf (robot description, URDF)
Before this commit: robot urdf_robot, 1 links, 0 joints
Links:
- link baseLink: geometry collision cylinder length=0.20 radius=0.06; visual cylinder length=0.20 radius=0.06

Commit message: minor mods

File: my_pybullet_envs/assets/cylinder.urdf (robot description, URDF)
Before this commit: robot urdf_robot, 1 links, 0 joints
Links:
- link baseLink: geometry collision cylinder length=0.20 radius=0.04; visual cylinder length=0.20 radius=0.04

Commit message: add shadow hand env

File: my_pybullet_envs/assets/cylinder.urdf (robot description, URDF)
Before this commit: robot urdf_robot, 1 links, 0 joints
Links:
- link baseLink: mass 2.5 -> 5.0

Commit message: 0118 reverts placing env

File: my_pybullet_envs/assets/cylinder.urdf (robot description, URDF)
Before this commit: robot urdf_robot, 1 links, 0 joints
Links:
- link baseLink: geometry collision cylinder length=0.18 radius=0.06; visual cylinder length=0.18 radius=0.06
