Commit message: new obj files

File: my_pybullet_envs/assets/box_small.urdf (robot description, URDF)
Before this commit: robot urdf_robot, 1 links, 0 joints
Links:
- link baseLink: geometry collision box size=0.05 0.05 0.13; visual box size=0.05 0.05 0.13

File: my_pybullet_envs/assets/cylinder.urdf (robot description, URDF)
Before this commit: robot urdf_robot, 1 links, 0 joints
Links:
- link baseLink: geometry collision cylinder length=0.18 radius=0.05; visual cylinder length=0.18 radius=0.05

File: my_pybullet_envs/assets/cylinder_small.urdf (robot description, URDF)
Before this commit: robot urdf_robot, 1 links, 0 joints
Links:
- link baseLink: geometry collision cylinder length=0.13 radius=0.04; visual cylinder length=0.13 radius=0.04

File: my_pybullet_envs/assets/sphere.urdf (robot description, URDF)
Before this commit: robot object, 1 links, 0 joints
Links:
- link baseLink: mass 5.0 -> 3.5; geometry collision sphere radius=0.045; visual sphere radius=0.045
