Commit message: mods grasping and placing

File: my_pybullet_envs/assets/tabletop.urdf (robot description, URDF)
Before this commit: robot tabletop, 1 links, 0 joints
Links:
- link baseLink: geometry collision box size=0.6 1.2 0.1; visual box size=0.6 1.2 0.1

Commit message: minor mods

File: my_pybullet_envs/assets/tabletop.urdf (robot description, URDF)
Before this commit: robot tabletop, 1 links, 0 joints
Links:
- link baseLink: geometry collision box size=0.6 2.0 0.1; visual box size=0.6 2.0 0.1
